Commit message: commit

File: urdf.xacro (robot description, xacro)
@@ -1,3 +1,4 @@
-<robot name="robot">
+<?xml version="1.0"?>
+<robot xmlns:xacro="http://www.ros.org/wiki/xacro" name="robot">
  <link name="base">
 	<visual>
@@ -70,4 +71,55 @@
 	</collision>
 </link>
+<xacro:macro name="xacro_name" params= "suffix_reflect">
+<xacro:xacro_name suffix="right" reflect="1"/>
+<link name="wheel_right">
+	<visual>
+		<origin xyz="-0.10 -0.4 0" rpy="-1.57 0 0"/>
+		<geometry>
+		<cylinder length="0.05" radius=".2"/>
+		</geometry>
+	</visual>
+	<collision>
+	<origin xyz="-0.10 -0.4 0" rpy="-1.57 0 0"/>
+	<geometry>
+	<cylinder radius="1" length="0.5"/>
+	</geometry>
+	</collision>
+</link>
+</xacro:macro>
+<xacro:macro name="xacro_name" params= "suffix_reflect">
+<xacro:xacro_name suffix="left" reflect="1"/>
+<link name="wheel_left">
+	<visual>
+		<origin xyz="-0.10 0.4 0" rpy="-1.57 0 0"/>
+		<geometry>
+		<cylinder length="0.05" radius=".2"/>
+		</geometry>
+	</visual>
+	<collision>
+	<origin xyz="-0.10 0.4 0" rpy="-1.57 0 0"/>
+	<geometry>
+	<cylinder radius="1" length="0.5"/>
+	</geometry>
+	</collision>
+</link>
+</xacro:macro>
+<xacro:macro name="xacro_name" params= "suffix_reflect">
+<xacro:xacro_name suffix="center" reflect="1"/>
+<link name="wheel_center">
+	<visual>
+		<origin xyz="0.10 0 0" rpy="-1.57 0 0"/>
+		<geometry>
+		<cylinder length="0.05" radius=".15"/>
+		</geometry>
+	</visual>
+	<collision>
+	<origin xyz="0.10 0 0" rpy="-1.57 0 0"/>
+	<geometry>
+	<cylinder radius="1" length="0.5"/>
+	</geometry>
+	</collision>
+</link>
+</xacro:macro>
 <joint name="base_vert_bottom_joint" type="floating">
 	<origin xyz="0.3158 -0.0021 0.5100" rpy="3.1355 -1.3045 0.0025"/>
@@ -90,3 +142,27 @@
 	<child link="laser_horiz"/>
 </joint>
+<xacro:macro name="xacro_name" params= "suffix_reflect">
+<xacro:xacro_name suffix="right" reflect="1"/>
+<joint name="base_wheel_right_joint" type="floating">
+	<origin xyz="-0.10 -0.4 0" rpy="-1.57 0 0"/>
+	<parent link="base"/>
+	<child link="wheel_right"/>
+</joint>
+</xacro:macro>
+<xacro:macro name="xacro_name" params= "suffix_reflect">
+<xacro:xacro_name suffix="left" reflect="1"/>
+<joint name="base_wheel_left_joint" type="floating">
+	<origin xyz="-0.10 0.4 0" rpy="-1.57 0 0"/>
+	<parent link="base"/>
+	<child link="wheel_left"/>
+</joint>
+</xacro:macro>
+<xacro:macro name="xacro_name" params= "suffix_reflect">
+<xacro:xacro_name suffix="center" reflect="1"/>
+<joint name="base_wheel_center_joint" type="floating">
+	<origin xyz="0.10 0 0" rpy="-1.57 0 0"/>
+	<parent link="base"/>
+	<child link="wheel_center"/>
+</joint>
+</xacro:macro>
 </robot>

Commit message: dkjf

File: urdf.xacro (robot description, xacro)
@@ -3,5 +3,5 @@
  <link name="base">
 	<visual>
-		<origin xyz="-.47 0 .99" rpy="0 0 0"/>
+		<origin xyz=".47 .39 .99" rpy="0 0 0"/>
 		<geometry>
 		<box size= ".94 .78 1.98"/>
@@ -9,5 +9,5 @@
    	</visual>
 	<collision>
-	<origin xyz="-.47 0 .99" rpy="0 0 0"/>
+	<origin xyz=".47 .39 .99" rpy="0 0 0"/>
 	<geometry>
 	<cylinder radius="1" length="0.5"/>

Commit message: commit

File: urdf.xacro (robot description, xacro)
@@ -17,5 +17,4 @@
 <link name="laser_vert_bottom">
 	<visual>
-		<origin xyz="0.3158 -0.0021 0.5100" rpy="3.1355 -1.3045 0.0025"/>
 		<geometry>
 		<box size= ".062 .062 0.087"/>
@@ -23,5 +22,4 @@
 	</visual>
 	<collision>
-	<origin xyz="0.3158 -0.0021 0.5100" rpy="3.1355 -1.3045 0.0025"/>
 	<geometry>
 	<cylinder radius="1" length="0.5"/>
@@ -31,5 +29,4 @@
 <link name="laser_vert_top_right">
 	<visual>
-		<origin xyz="0.2978 -0.1450 1.8451" rpy="-1.1760 0.6313 -1.9377"/>
 		<geometry>
 		<box size= ".062 .062 0.087"/>
@@ -37,5 +34,4 @@
 	</visual>
 	<collision>
-	<origin xyz="0.2978 -0.1450 1.8451" rpy="-1.1760 0.6313 -1.9377"/>
 	<geometry>
 	<cylinder radius="1" length="0.5"/>
@@ -45,5 +41,4 @@
 <link name="laser_vert_top_left">
 	<visual>
-		<origin xyz="0.2997 0.1531 1.8443" rpy="1.1780 0.6198 1.9560"/>
 		<geometry>
 		<box size= ".062 .062 0.087"/>
@@ -51,5 +46,4 @@
 	</visual>
 	<collision>
-	<origin xyz="0.2997 0.1531 1.8443" rpy="1.1780 0.6198 1.9560"/>
 	<geometry>
 	<cylinder radius="1" length="0.5"/>
@@ -59,5 +53,4 @@
 <link name="laser_horiz">
 	<visual>
-		<origin xyz="0.2325 .0001 1.9201" rpy="-0.0012 0.1146 -0.0015"/>
 		<geometry>
 		<cylinder length=".072" radius=".052"/>
@@ -65,5 +58,4 @@
 	</visual>
 	<collision>
-	<origin xyz="0.2325 .0001 1.9201" rpy="-0.0012 0.1146 -0.0015"/>
 	<geometry>
 	<cylinder radius="1" length="0.5"/>
@@ -71,9 +63,6 @@
 	</collision>
 </link>
-<xacro:macro name="xacro_name" params= "suffix_reflect">
-<xacro:xacro_name suffix="right" reflect="1"/>
 <link name="wheel_right">
 	<visual>
-		<origin xyz="-0.10 -0.4 0" rpy="-1.57 0 0"/>
 		<geometry>
 		<cylinder length="0.05" radius=".2"/>
@@ -81,5 +70,4 @@
 	</visual>
 	<collision>
-	<origin xyz="-0.10 -0.4 0" rpy="-1.57 0 0"/>
 	<geometry>
 	<cylinder radius="1" length="0.5"/>
@@ -87,10 +75,7 @@
 	</collision>
 </link>
-</xacro:macro>
-<xacro:macro name="xacro_name" params= "suffix_reflect">
-<xacro:xacro_name suffix="left" reflect="1"/>
+<xacro:macro name="xacro_name" params= "suffix reflect">
 <link name="wheel_left">
 	<visual>
-		<origin xyz="-0.10 0.4 0" rpy="-1.57 0 0"/>
 		<geometry>
 		<cylinder length="0.05" radius=".2"/>
@@ -105,9 +90,7 @@
 </link>
 </xacro:macro>
-<xacro:macro name="xacro_name" params= "suffix_reflect">
-<xacro:xacro_name suffix="center" reflect="1"/>
+<xacro:xacro_name suffix="left" reflect="1"/>
 <link name="wheel_center">
 	<visual>
-		<origin xyz="0.10 0 0" rpy="-1.57 0 0"/>
 		<geometry>
 		<cylinder length="0.05" radius=".15"/>
@@ -115,5 +98,4 @@
 	</visual>
 	<collision>
-	<origin xyz="0.10 0 0" rpy="-1.57 0 0"/>
 	<geometry>
 	<cylinder radius="1" length="0.5"/>
@@ -121,36 +103,31 @@
 	</collision>
 </link>
-</xacro:macro>
-<joint name="base_vert_bottom_joint" type="floating">
+<joint name="base_vert_bottom_joint" type="fixed">
 	<origin xyz="0.3158 -0.0021 0.5100" rpy="3.1355 -1.3045 0.0025"/>
 	<parent link="base"/>
 	<child link="laser_vert_bottom"/>
 </joint>
-<joint name="base_vert_top_right_joint" type="floating">
+<joint name="base_vert_top_right_joint" type="fixed">
 	<origin xyz="0.2978 -0.1450 1.8451" rpy="-1.1760 0.6313 -1.9377"/>
 	<parent link="base"/>
 	<child link="laser_vert_top_right"/>
 </joint>
-<joint name="base_vert_top_left_joint" type="floating">
+<joint name="base_vert_top_left_joint" type="fixed">
 	<origin xyz="0.2997 0.1531 1.8443" rpy="1.1780 0.6198 1.9560"/>
 	<parent link="base"/>
 	<child link="laser_vert_top_left"/>
 </joint>
-<joint name="base_horiz_joint" type="floating">
+<joint name="base_horiz_joint" type="fixed">
 	<origin xyz="0.2325 .0001 1.9201" rpy="-0.0012 0.1146 -0.0015"/>
 	<parent link="base"/>
 	<child link="laser_horiz"/>
 </joint>
-<xacro:macro name="xacro_name" params= "suffix_reflect">
-<xacro:xacro_name suffix="right" reflect="1"/>
-<joint name="base_wheel_right_joint" type="floating">
+<joint name="base_wheel_right_joint" type="fixed">
 	<origin xyz="-0.10 -0.4 0" rpy="-1.57 0 0"/>
 	<parent link="base"/>
 	<child link="wheel_right"/>
 </joint>
-</xacro:macro>
-<xacro:macro name="xacro_name" params= "suffix_reflect">
-<xacro:xacro_name suffix="left" reflect="1"/>
-<joint name="base_wheel_left_joint" type="floating">
+<xacro:macro name="xacro_left" params= "suffix reflect">
+<joint name="base_wheel_left_joint" type="fixed">
 	<origin xyz="-0.10 0.4 0" rpy="-1.57 0 0"/>
 	<parent link="base"/>
@@ -158,11 +135,9 @@
 </joint>
 </xacro:macro>
-<xacro:macro name="xacro_name" params= "suffix_reflect">
-<xacro:xacro_name suffix="center" reflect="1"/>
-<joint name="base_wheel_center_joint" type="floating">
+<xacro:xacro_left suffix="left" reflect="1"/>
+<joint name="base_wheel_center_joint" type="fixed">
 	<origin xyz="0.10 0 0" rpy="-1.57 0 0"/>
 	<parent link="base"/>
 	<child link="wheel_center"/>
 </joint>
-</xacro:macro>
 </robot>

Commit message: commit

File: urdf.xacro (robot description, xacro)
@@ -63,4 +63,5 @@
 	</collision>
 </link>
+<xacro:macro name="xacro_right" params= "suffix reflect">
 <link name="wheel_right">
 	<visual>
@@ -75,5 +76,7 @@
 	</collision>
 </link>
-<xacro:macro name="xacro_name" params= "suffix reflect">
+</xacro:macro>
+<xacro:xacro_right suffix="right" reflect="-1"/>
+<xacro:macro name="xacro_left" params= "suffix reflect">
 <link name="wheel_left">
 	<visual>
@@ -90,5 +93,5 @@
 </link>
 </xacro:macro>
-<xacro:xacro_name suffix="left" reflect="1"/>
+<xacro:xacro_left suffix="left" reflect="1"/>
 <link name="wheel_center">
 	<visual>
@@ -123,4 +126,5 @@
 	<child link="laser_horiz"/>
 </joint>
+<xacro:macro name="xacro_name" params= "suffix reflect">
 <joint name="base_wheel_right_joint" type="fixed">
 	<origin xyz="-0.10 -0.4 0" rpy="-1.57 0 0"/>
@@ -128,5 +132,7 @@
 	<child link="wheel_right"/>
 </joint>
-<xacro:macro name="xacro_left" params= "suffix reflect">
+</xacro:macro>
+<xacro:xacro_name suffix="right" reflect="-1"/>
+<xacro:macro name="xacro_left2" params= "suffix reflect">
 <joint name="base_wheel_left_joint" type="fixed">
 	<origin xyz="-0.10 0.4 0" rpy="-1.57 0 0"/>
@@ -135,5 +141,5 @@
 </joint>
 </xacro:macro>
-<xacro:xacro_left suffix="left" reflect="1"/>
+<xacro:xacro_left2 suffix="left" reflect="1"/>
 <joint name="base_wheel_center_joint" type="fixed">
 	<origin xyz="0.10 0 0" rpy="-1.57 0 0"/>

Commit message: commit

File: urdf.xacro (robot description, xacro)
@@ -127,6 +127,6 @@
 </joint>
 <xacro:macro name="xacro_name" params= "suffix reflect">
-<joint name="base_wheel_right_joint" type="fixed">
-	<origin xyz="-0.10 -0.4 0" rpy="-1.57 0 0"/>
+<joint name="base_wheel_right_joint" type="continuous">
+	<origin xyz="-0.10 ${reflect * 0.4} 0" rpy="-1.57 0 0"/>
 	<parent link="base"/>
 	<child link="wheel_right"/>
@@ -135,5 +135,5 @@
 <xacro:xacro_name suffix="right" reflect="-1"/>
 <xacro:macro name="xacro_left2" params= "suffix reflect">
-<joint name="base_wheel_left_joint" type="fixed">
+<joint name="base_wheel_left_joint" type="continuous">
 	<origin xyz="-0.10 0.4 0" rpy="-1.57 0 0"/>
 	<parent link="base"/>
@@ -142,5 +142,5 @@
 </xacro:macro>
 <xacro:xacro_left2 suffix="left" reflect="1"/>
-<joint name="base_wheel_center_joint" type="fixed">
+<joint name="base_wheel_center_joint" type="continuous">
 	<origin xyz="0.10 0 0" rpy="-1.57 0 0"/>
 	<parent link="base"/>

File: urdf_from_xacro.urdf (robot description, URDF)
Before this commit: robot robot, 8 links, 7 joints
Joints:
- joint base_wheel_center_joint: type fixed -> continuous
- joint base_wheel_left_joint: type fixed -> continuous
- joint base_wheel_right_joint: type fixed -> continuous
